File: templates/kicad/T44-10/T44-10.kicad_pcb (KiCad board)
At the start: 2 copper layers, 4 x 4 mm, 10 parts

Commit message: Adding pin numbers to pads in template files.
Another way to have iterating pads would have been to add one N-pin header, but that would lock all the pads to one location on the schematic, not ideal. The other would have been to create 22 custom schematic pin symbols, iterating the pad numbers in there. But that would duplicate pad structures. Much more elegant (imho) to have the pads be labelled in the user comments layer.
Other:
- board text added: "P1"
- board text added: "P10"
- board text added: "P2"
- board text added: "P3"
- board text added: "P4"
- board text added: "P5"
- board text added: "P6"
- board text added: "P7"
- board text added: "P8"
- board text added: "P9"
